Commit message: Link for the camera mounted on top of R1's head

File: R1SN003/cer.urdf (robot description, URDF)
Before this commit: robot SIM_CER_ROBOT, 61 links, 60 joints
Links:
- added link external_depth_center
Joints:
- added joint external_depth_center_fixed_joint: type fixed, parent depth_center, child external_depth_center, origin xyz=0.0 0 0.15 rpy=0 0 0
